File: pcb/digital_clock_v1/digital_clock_v1.kicad_pcb (KiCad board)
At the start: 2 copper layers, 38 parts, among them J1 USB_B_Mini, T1 terminal_3x1, T2 terminal_8x1, T3 terminal_3x1, U1 DS3231, U2 SD2405AL, U3 CA56-12SRWA, U4 ATmega328P-A, U5 8X8PADS, Y1 Crystal-Device_SMD_4pins_16MHz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

Commit message: Add pcb design, not yet ready
Parts:
- added H1: MountingHole, Luciebox:MountingHole_4.3mm_M4, F.Cu at (25.4, 66.0)
- added H2: MountingHole, Luciebox:MountingHole_4.3mm_M4, F.Cu at (97.8, 67.3)
- added H3: MountingHole, Luciebox:MountingHole_4.3mm_M4, F.Cu at (99.1, 141.0)
- added H4: MountingHole, Luciebox:MountingHole_4.3mm_M4, F.Cu at (14.0, 142.2)
- U3: footprint Luciebox:CA56-12SRWA -> Lucieboxv3:CA56-12SRWA
- moved T3 164.3 mm to (57.1, 141.0), turned to -90 degrees
- moved S9 132.2 mm to (64.9, 139.7), turned to -90 degrees

Commit message: PCB Send out v1
Parts:
- removed S5, S6, S7, S8: button_laz16-11, Luciebox:button_LAZ16-11_big_holes
- removed U2: SD2405AL, digital_clock:SD2405AL
- added U6: 8X8PADS, Luciebox:8X8PADS_100mil, F.Cu at (11.8, 37.7)
- added Upsidedown1: CA56-12SRWA, Lucieboxv3:CA56-12SRWA, F.Cu at (40.4, 46.5)
- BZ1, J1: moved to B.Cu
- U3: moved to F.Cu
- U5: value 8X8PADS -> CA56-12SRWA; footprint Luciebox:8X8PADS_100mil -> Lucieboxv3:CA56-12SRWA
- moved H4 151.0 mm to (78.0, 5.50)
- moved S1 124.9 mm to (27.4, 8.64), turned to -90 degrees
- moved T3 118.9 mm to (86.6, 25.8), turned to 180 degrees
- moved S4 118.1 mm to (66.8, 8.64), turned to -90 degrees
- moved S2 114.6 mm to (40.5, 8.64), turned to -90 degrees
- moved S3 112.2 mm to (53.6, 8.64), turned to -90 degrees
- moved S9 111.8 mm to (84.0, 29.5), turned to 180 degrees
- moved C4 106.8 mm to (15.4, 22.5)
- moved C3 105.2 mm to (15.4, 16.2)
- moved C2 105.0 mm to (5.59, 20.0)
- moved H2 102.8 mm to (16.0, 5.00)
- moved D1 102.7 mm to (15.4, 25.7)
- moved R1 102.1 mm to (8.64, 25.9)
- moved BZ1 97.5 mm to (78.5, 18.5), turned to 180 degrees
- moved J1 93.8 mm to (93.4, 19.5), turned to 180 degrees
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Connections:
- T2 pad 1: unconnected-(T2-Pad1) -> VCC
- T2 pad 2: unconnected-(T2-Pad2) -> /A5(SCL)
- T2 pad 3: unconnected-(T2-Pad3) -> /A4(SDA)
- U5 pad 1: VCC -> /0(Rx)
- U5 pad 10: Net-(U5-Pad10) -> /13(SCK)
- U5 pad 11: Net-(U5-Pad10) -> /12(MISO)
- U5 pad 12: Net-(U5-Pad10) -> Net-(R9-Pad1)
- U5 pad 2: VCC -> /3(PWM)
- U5 pad 3: VCC -> /4
- U5 pad 4: VCC -> /11(PWM-MOSI)
- U5 pad 5: VCC -> /7
- U5 pad 6: VCC -> Net-(R6-Pad1)
- U5 pad 7: VCC -> /8
- U5 pad 8: VCC -> Net-(R7-Pad1)
- U5 pad 9: Net-(U5-Pad10) -> Net-(R8-Pad1)
Routing:
- net VCC: track 0.00 -> 192.4 mm, vias 0 -> 4
- net Net-(C1-Pad2): track 0.00 -> 119.6 mm, vias 0 -> 1
- net /2: track 0.00 -> 84.9 mm, vias 0 -> 2
- net /A3: track 0.00 -> 81.1 mm, vias 0 -> 2
- net /A0: track 0.00 -> 75.4 mm
- net /A2: track 0.00 -> 72.0 mm, vias 0 -> 2
- net /A1: track 0.00 -> 69.6 mm, vias 0 -> 2
- net /13(SCK): track 0.00 -> 67.7 mm, vias 0 -> 1
- net /0(Rx): track 0.00 -> 64.2 mm, vias 0 -> 1
- net /8: track 0.00 -> 63.9 mm, vias 0 -> 1
- net /12(MISO): track 0.00 -> 63.7 mm, vias 0 -> 1
- net /A4(SDA): track 0.00 -> 63.7 mm, vias 0 -> 1
- net /A5(SCL): track 0.00 -> 61.9 mm, vias 0 -> 1
- net Net-(R6-Pad1): track 0.00 -> 56.6 mm, vias 0 -> 1
- net Net-(R8-Pad1): track 0.00 -> 53.7 mm, vias 0 -> 1
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- added copper zone on B.Cu, net GND
- added copper zone on F.Cu, net GND
Other:
- board outline added: 93.5 x 61.5 mm
- board text added: "+"
- board text added: "-"
- board text added: "Alarm Clock v1.0 2022-11 ameije.com Project for Lucie and Ramses by Uncle Low-D"
- board text added: "ESC"
- board text added: "OK"
