File: pcb/digital_clock_v1/digital_clock_v1.kicad_sch (KiCad schematic)
At the start: 42 parts, among them J1 USB_B_Mini, T1 terminal_3x1, T2 terminal_8x1, T3 terminal_3x1, U1 DS3231, U2 SD2405AL, U3 CA56-12SRWA, U4 ATmega328P-A, U5 8X8PADS, Y1 Crystal-Device_SMD_4pins_16MHz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

Commit message: Add pcb design, not yet ready
Parts:
- U3: footprint Luciebox:CA56-12SRWA -> Lucieboxv3:CA56-12SRWA
Changed lines of the file:
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@@
     (property "Reference" "U3" (id 0) (at 76.2 71.9582 0))
     (property "Value" "CA56-12SRWA" (id 1) (at 76.2 74.2696 0))
-    (property "Footprint" "Luciebox:CA56-12SRWA" (id 2) (at 76.2 104.14 0)
+    (property "Footprint" "Lucieboxv3:CA56-12SRWA" (id 2) (at 76.2 104.14 0)
       (effects (font (size 1.27 1.27)) hide)
     )
@@
     )
     (path "/a1ca69cd-817d-4f8b-ab26-4c311a7c46df"
-      (reference "U3") (unit 1) (value "CA56-12SRWA") (footprint "Luciebox:CA56-12SRWA")
+      (reference "U3") (unit 1) (value "CA56-12SRWA") (footprint "Lucieboxv3:CA56-12SRWA")
     )
     (path "/dd927aef-0d69-4bac-b16b-5b63d94e7773"

Commit message: PCB Send out v1
Parts:
- removed S5, S6, S7, S8: button_laz16-11, Luciebox:button_LAZ16-11_big_holes, symbol Luciebox_components:button_laz16-11
- removed U2: SD2405AL, digital_clock:SD2405AL, symbol digital_clock:SD2405AL
- added U5, Upsidedown1: CA56-12SRWA, Lucieboxv3:CA56-12SRWA, symbol Luciebox_components:4digit_7segments_common_anode_CA56-12SRWA
- renumbered U5 to U6
Connections:
- net 0(Rx): now also U5.1 (e), Upsidedown1.10 (f)
- net 11(PWM-MOSI): now also U5.4 (c), Upsidedown1.7 (b)
- net 12(MISO): now also U5.11 (a), Upsidedown1.2 (d)
- net 13(SCK): now also U5.10 (f), Upsidedown1.1 (e)
- net 3(PWM): now also U5.2 (d), Upsidedown1.11 (a)
- net 4: now also U5.3 (DPX), Upsidedown1.3 (DPX)
- net 7: now also U5.5 (g), Upsidedown1.5 (g)
- net 8: now also U5.7 (b), Upsidedown1.4 (c)
- net A4(SDA): now also T2.3
- net A5(SCL): now also T2.2
- net VCC: now also T2.1
- net at R8.1, U3.9 (CA2): now also U5.9 (CA2), Upsidedown1.9 (CA2)
- net at R7.1, U3.8 (CA3): now also U5.8 (CA3), Upsidedown1.8 (CA3)
- net at R9.1, U3.12 (CA1): now also U5.12 (CA1), Upsidedown1.12 (CA1)
- net at R6.1, U3.6 (CA4): now also U5.6 (CA4), Upsidedown1.6 (CA4)
Other:
- moved on the sheet: BZ1, H1, H2, H3, H4, R6, R7, R8, R9, S9, T2, T3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
