File: pcb/digital_clock_v2/digital_clock_v2.kicad_pcb (KiCad board)
At the start: 2 copper layers, 93.5 x 49.5 mm, 36 parts, among them J1 USB_B_Mini, J2 USB_B_Mini, T1 terminal_3x1, T2 terminal_8x1, T3 terminal_3x1, U1 DS3231, U3 CA56-12SRWA, U4 ATmega328P-A, Y1 Crystal-Device_SMD_4pins_16MHz, Y2 16MHz

Commit message: Finish v2 pcb wiring
Parts:
- removed H2, H4: MountingHole, Luciebox:MountingHole_4.3mm_M4
- moved C2 2.95 mm to (6.99, 17.8), turned to -90 degrees
- moved T1 1.40 mm to (62.6, 59.7), turned to 0 degrees
- moved C3 0.34 mm to (14.8, 38.1)
Routing:
- net VCC: track 0.00 -> 158.9 mm
- net GND: track 0.00 -> 134.0 mm, vias 0 -> 42
- net Net-(C1-Pad2): track 0.00 -> 129.9 mm, vias 0 -> 3
- net /A4(SDA): track 0.00 -> 73.2 mm, vias 0 -> 3
- net /A5(SCL): track 0.00 -> 67.0 mm, vias 0 -> 4
- net /0(Rx): track 0.00 -> 59.5 mm, vias 0 -> 2
- net /A0: track 0.00 -> 57.1 mm, vias 0 -> 1
- net /9(PWM): track 0.00 -> 43.3 mm, vias 0 -> 2
- net Net-(R6-Pad1): track 0.00 -> 42.1 mm
- net Net-(R5-Pad1): track 0.00 -> 39.7 mm, vias 0 -> 1
- net /A1: track 0.00 -> 38.9 mm, vias 0 -> 2
- net /6(PWM): track 0.00 -> 36.9 mm, vias 0 -> 2
- net /10(PWM-SS): track 0.00 -> 33.6 mm, vias 0 -> 4
- net /5(PWM): track 0.00 -> 31.3 mm
- net Net-(R9-Pad1): track 0.00 -> 29.9 mm, vias 0 -> 1
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Other:
- outline, holes or cut-outs redrawn
- board text added: "Alarm Clock v2.0 2023-02 ameije.com Project for Lucie and Ramses by Uncle Low-D"
- board text removed: "Alarm Clock v1.0 2022-11 ameije.com Project for Lucie and Ramses by Uncle Low-D"

Commit message: Correct button positions
Parts:
- moved S5 4.66 mm to (18.0, 22.3)
- moved S6 4.66 mm to (37.0, 22.3)
- moved S7 4.66 mm to (56.0, 22.3)
- moved S8 4.66 mm to (75.0, 22.3)
Routing:
- net Net-(C1-Pad2): track 129.9 -> 110.4 mm, vias 3 -> 2
- net /A3: track 22.1 -> 26.8 mm
- net /A2: track 21.9 -> 26.6 mm
- net /A1: track 38.9 -> 43.5 mm
- net /2: track 23.0 -> 27.3 mm
