File: pcb/digital_clock_v2/digital_clock_v2.kicad_sch (KiCad schematic)
At the start: 36 parts, among them J1 USB_B_Mini, J2 USB_B_Mini, T1 terminal_3x1, T2 terminal_8x1, T3 terminal_3x1, U1 DS3231, U3 CA56-12SRWA, U4 ATmega328P-A, Y1 Crystal-Device_SMD_4pins_16MHz, Y2 16MHz

Commit message: Finish v2 pcb wiring
Parts:
- removed H2, H4: MountingHole, Luciebox:MountingHole_4.3mm_M4, symbol digital_clock:MountingHole
Changed lines of the file:
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@@
     (effects (font (size 1.27 1.27)) (justify left bottom))
-  )
-  (symbol (lib_id "digital_clock:MountingHole") (at 156.21 191.77 0) (unit 1)
-    (in_bom yes) (on_board yes) (fields_autoplaced)
-    (property "Reference" "H4" (id 0) (at 158.75 190.4999 0)
-      (effects (font (size 1.27 1.27)) (justify left))
-    )
-    (property "Value" "MountingHole" (id 1) (at 158.75 193.0399 0)
-      (effects (font (size 1.27 1.27)) (justify left))
-    )
-    (property "Footprint" "Luciebox:MountingHole_4.3mm_M4" (id 2) (at 156.21 191.77 0)
-      (effects (font (size 1.27 1.27)) hide)
-    )
-    (property "Datasheet" "~" (id 3) (at 156.21 191.77 0)
-      (effects (font (size 1.27 1.27)) hide)
-    )
   )
   (symbol (lib_id "jlcpcb-basic-capacitor:0603,100nF,50V,X7R ") (at 246.38 38.1 180) (unit 1)
@@
     (pin "2")
     (pin "3")
-  )
-  (symbol (lib_id "digital_clock:MountingHole") (at 156.21 180.34 0) (unit 1)
-    (in_bom yes) (on_board yes) (fields_autoplaced)
-    (property "Reference" "H2" (id 0) (at 158.75 179.0699 0)
-      (effects (font (size 1.27 1.27)) (justify left))
-    )
-    (property "Value" "MountingHole" (id 1) (at 158.75 181.6099 0)
-      (effects (font (size 1.27 1.27)) (justify left))
-    )
-    (property "Footprint" "Luciebox:MountingHole_4.3mm_M4" (id 2) (at 156.21 180.34 0)
-      (effects (font (size 1.27 1.27)) hide)
-    )
-    (property "Datasheet" "~" (id 3) (at 156.21 180.34 0)
-      (effects (font (size 1.27 1.27)) hide)
-    )
   )
   (symbol (lib_id "Luciebox_components:Crystal-Device") (at 261.62 87.63 270) (unit 1)
@@
       (reference "H1") (unit 1) (value "MountingHole") (footprint "Luciebox:MountingHole_4.3mm_M4")
     )
-    (path "/4cc7c4ed-f40f-4be8-a362-8f14caa2d011"
-      (reference "H2") (unit 1) (value "MountingHole") (footprint "Luciebox:MountingHole_4.3mm_M4")
-    )
     (path "/2ff5e44d-1c39-4cc7-9a27-d0df9a66cdaf"
       (reference "H3") (unit 1) (value "MountingHole") (footprint "Luciebox:MountingHole_4.3mm_M4")
     )
-    (path "/0024a8c6-9f6d-449f-b8b7-4d233b38f166"
-      (reference "H4") (unit 1) (value "MountingHole") (footprint "Luciebox:MountingHole_4.3mm_M4")
-    )
     (path "/086877e6-a6d1-4b60-b3a6-6372a409a809"

Commit message: Correct button positions
Changed lines of the file:
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@@
   (junction (at 248.92 80.01) (diameter 0) (color 0 0 0 0)
   )
-  (junction (at 45.72 44.45) (diameter 0) (color 0 0 0 0)
-  )
-  (junction (at 25.4 44.45) (diameter 0) (color 0 0 0 0)
-  )
   (junction (at 198.12 68.58) (diameter 0) (color 0 0 0 0)
   )
@@
   (junction (at 257.81 62.23) (diameter 0) (color 0 0 0 0)
   )
-  (junction (at 101.6 44.45) (diameter 0) (color 0 0 0 0)
-  )
   (junction (at 233.68 74.93) (diameter 0) (color 0 0 0 0)
   )
@@
   (junction (at 251.46 71.12) (diameter 0) (color 0 0 0 0)
   )
-  (junction (at 64.77 44.45) (diameter 0) (color 0 0 0 0)
-  )
   (junction (at 255.27 114.3) (diameter 0) (color 0 0 0 0)
   )
@@
   (junction (at 219.71 114.3) (diameter 0) (color 0 0 0 0)
   )
-  (junction (at 156.21 45.72) (diameter 0) (color 0 0 0 0)
-  )
   (junction (at 262.89 50.8) (diameter 0) (color 0 0 0 0)
   )
   (junction (at 236.22 43.18) (diameter 0) (color 0 0 0 0)
   )
-  (junction (at 83.82 44.45) (diameter 0) (color 0 0 0 0)
-  )
   (junction (at 236.22 40.64) (diameter 0) (color 0 0 0 0)
   )
@@
   (junction (at 242.57 71.12) (diameter 0) (color 0 0 0 0)
   )
-  (junction (at 120.65 44.45) (diameter 0) (color 0 0 0 0)
-  )
   (junction (at 257.81 71.12) (diameter 0) (color 0 0 0 0)
   )
@@
   (junction (at 205.74 43.18) (diameter 0) (color 0 0 0 0)
   )
-  (junction (at 134.62 45.72) (diameter 0) (color 0 0 0 0)
-  )
   (wire (pts (xy 106.68 175.26) (xy 125.73 175.26))
     (stroke (width 0) (type default) (color 0 0 0 0))
@@
     (stroke (width 0) (type default) (color 0 0 0 0))
   )
-  (wire (pts (xy 68.58 44.45) (xy 64.77 44.45))
-    (stroke (width 0) (type default) (color 0 0 0 0))
-  )
   (wire (pts (xy 27.94 175.26) (xy 27.94 171.45))
     (stroke (width 0) (type default) (color 0 0 0 0))
@@
     (stroke (width 0) (type default) (color 0 0 0 0))
   )
-  (wire (pts (xy 104.14 44.45) (xy 101.6 44.45))
-    (stroke (width 0) (type default) (color 0 0 0 0))
-  )
   (wire (pts (xy 245.11 78.74) (xy 247.65 78.74))
     (stroke (width 0) (type default) (color 0 0 0 0))
@@
     (stroke (width 0) (type default) (color 0 0 0 0))
   )
-  (wire (pts (xy 139.7 45.72) (xy 134.62 45.72))
-    (stroke (width 0) (type default) (color 0 0 0 0))
-  )
   (wire (pts (xy 33.02 195.58) (xy 45.72 195.58))
     (stroke (width 0) (type default) (color 0 0 0 0))
@@
     (stroke (width 0) (type default) (color 0 0 0 0))
   )
-  (wire (pts (xy 114.3 44.45) (xy 120.65 44.45))
-    (stroke (width 0) (type default) (color 0 0 0 0))
-  )
   (wire (pts (xy 186.69 25.4) (xy 186.69 38.1))
     (stroke (width 0) (type default) (color 0 0 0 0))
@@
     (stroke (width 0) (type default) (color 0 0 0 0))
   )
-  (wire (pts (xy 149.86 45.72) (xy 156.21 45.72))
-    (stroke (width 0) (type default) (color 0 0 0 0))
-  )
   (wire (pts (xy 29.21 96.52) (xy 41.91 96.52))
     (stroke (width 0) (type default) (color 0 0 0 0))
@@
     (stroke (width 0) (type default) (color 0 0 0 0))
   )
-  (wire (pts (xy 30.48 44.45) (xy 25.4 44.45))
-    (stroke (width 0) (type default) (color 0 0 0 0))
-  )
   (wire (pts (xy 255.27 114.3) (xy 260.35 114.3))
     (stroke (width 0) (type default) (color 0 0 0 0))
@@
     (stroke (width 0) (type default) (color 0 0 0 0))
   )
-  (wire (pts (xy 78.74 44.45) (xy 83.82 44.45))
-    (stroke (width 0) (type default) (color 0 0 0 0))
-  )
   (wire (pts (xy 120.65 34.29) (xy 120.65 44.45))
     (stroke (width 0) (type default) (color 0 0 0 0))
@@
     (stroke (width 0) (type default) (color 0 0 0 0))
   )
-  (wire (pts (xy 40.64 44.45) (xy 45.72 44.45))
-    (stroke (width 0) (type default) (color 0 0 0 0))
-  )
