File: pcb/digital_clock_v3/digital_clock_v3.kicad_sch (KiCad schematic)
At the start: 34 parts, among them J1 USB_B_Mini, J2 USB_B_Mini, T1 terminal_3x1, T2 terminal_8x1, T3 terminal_3x1, U1 DS3231, U3 CA56-12SRWA, U4 ATmega328P-A, Y1 Crystal-Device_SMD_4pins_16MHz, Y2 16MHz

Commit message: Create v3 pcb
Parts:
- R1: value high current 220ohm worked ok in v2 -> high current
Connections:
- net 11(PWM-MOSI): now also T2.3
- net 12(MISO): now also T2.2
- net 13(SCK): now also T2.1
- net A4(SDA): no longer T2.3
- net A5(SCL): no longer T2.2
- net VCC: no longer T2.1
Changed lines of the file:
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@@
   (junction (at 255.27 114.3) (diameter 0) (color 0 0 0 0)
   )
-  (junction (at 256.54 124.46) (diameter 0) (color 0 0 0 0)
-  )
   (junction (at 205.74 45.72) (diameter 0) (color 0 0 0 0)
   )
@@
     (stroke (width 0) (type default) (color 0 0 0 0))
   )
-  (wire (pts (xy 256.54 124.46) (xy 219.71 124.46))
-    (stroke (width 0) (type default) (color 0 0 0 0))
-  )
   (wire (pts (xy 261.62 83.82) (xy 261.62 73.66))
     (stroke (width 0) (type default) (color 0 0 0 0))
@@
     (stroke (width 0) (type default) (color 0 0 0 0))
   )
-  (wire (pts (xy 255.27 132.08) (xy 274.32 132.08))
-    (stroke (width 0) (type default) (color 0 0 0 0))
-  )
   (wire (pts (xy 207.01 30.48) (xy 210.82 30.48))
     (stroke (width 0) (type default) (color 0 0 0 0))
@@
     (stroke (width 0) (type default) (color 0 0 0 0))
   )
-  (wire (pts (xy 255.27 114.3) (xy 255.27 132.08))
-    (stroke (width 0) (type default) (color 0 0 0 0))
-  )
   (wire (pts (xy 261.62 91.44) (xy 248.92 91.44))
     (stroke (width 0) (type default) (color 0 0 0 0))
@@
     (stroke (width 0) (type default) (color 0 0 0 0))
   )
-  (wire (pts (xy 256.54 99.06) (xy 256.54 124.46))
-    (stroke (width 0) (type default) (color 0 0 0 0))
-  )
   (wire (pts (xy 252.73 119.38) (xy 274.32 119.38))
     (stroke (width 0) (type default) (color 0 0 0 0))
@@
     (stroke (width 0) (type default) (color 0 0 0 0))
   )
-  (wire (pts (xy 274.32 127) (xy 245.11 127))
-    (stroke (width 0) (type default) (color 0 0 0 0))
-  )
   (wire (pts (xy 134.62 45.72) (xy 129.54 45.72))
     (stroke (width 0) (type default) (color 0 0 0 0))
@@
     (stroke (width 0) (type default) (color 0 0 0 0))
   )
-  (wire (pts (xy 274.32 129.54) (xy 245.11 129.54))
-    (stroke (width 0) (type default) (color 0 0 0 0))
-  )
   (wire (pts (xy 93.98 44.45) (xy 93.98 45.72))
     (stroke (width 0) (type default) (color 0 0 0 0))
@@
     (stroke (width 0) (type default) (color 0 0 0 0))
   )
-  (wire (pts (xy 274.32 124.46) (xy 256.54 124.46))
+  (wire (pts (xy 219.71 124.46) (xy 274.32 124.46))
     (stroke (width 0) (type default) (color 0 0 0 0))
   )
@@
     (effects (font (size 1.27 1.27)) (justify left bottom))
   )
-  (label "A4(SDA)" (at 245.11 127 180)
+  (label "13(SCK)" (at 274.32 132.08 180)
     (effects (font (size 1.27 1.27)) (justify right bottom))
   )
@@
     (effects (font (size 1.27 1.27)) (justify left bottom))
   )
-  (label "A5(SCL)" (at 245.11 129.54 180)
-    (effects (font (size 1.27 1.27)) (justify right bottom))
-  )
   (label "6(PWM)" (at 132.08 119.38 270)
     (effects (font (size 1.27 1.27)) (justify right bottom))
@@
     (effects (font (size 1.27 1.27)) (justify right bottom))
   )
+  (label "12(MISO)" (at 274.32 129.54 180)
+    (effects (font (size 1.27 1.27)) (justify right bottom))
+  )
   (label "9(PWM)" (at 213.36 78.74 0)
     (effects (font (size 1.27 1.27)) (justify left bottom))
@@
   (label "A5(SCL)" (at 229.87 30.48 0)
     (effects (font (size 1.27 1.27)) (justify left bottom))
+  )
+  (label "11(PWM-MOSI)" (at 274.32 127 180)
+    (effects (font (size 1.27 1.27)) (justify right bottom))
   )
   (label "1(Tx)" (at 252.73 119.38 180)
@@
       (effects (font (size 1.27 1.27)) (justify right))
     )
-    (property "Value" "high current 220ohm worked ok in v2" (id 1) (at 265.43 33.0199 0)
+    (property "Value" "high current" (id 1) (at 265.43 33.0199 0)
       (effects (font (size 1.27 1.27)) (justify right))
     )
@@
     )
     (path "/7f39a742-ce87-4808-9c57-866a2f4eb45a"
-      (reference "R1") (unit 1) (value "high current 220ohm worked ok in v2") (footprint "R_0603_1608Metric")
+      (reference "R1") (unit 1) (value "high current") (footprint "R_0603_1608Metric")
     )
     (path "/89b08bfd-462e-4897-9706-f2900ad93b29"
